File: hardware/VU meter PP4/VU meter PP4.kicad_sch (KiCad schematic)
At the start: 34 parts, among them J1 Conn_01x06_Pin, J2 Conn_01x03_Pin, J3 Conn_01x03_Pin, J4 Conn_01x04_Pin, J5 Conn_01x20_Socket, U1 KR1534PP4, U2 LM318J

Commit message: Cosmetic cleanup in schematics, add schematic PDF exports
Other:
- title: (none) -> VFD VU Meter Board
- moved on the sheet: H1, H2, H3, H4
Changed lines of the file:
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@@
 	(generator_version "9.0")
 	(paper "A4")
+	(title_block
+		(title "VFD VU Meter Board")
+	)
 	(junction
 		(at 93.98 77.47)
@@
 	(symbol
 		(lib_id "Mechanical:MountingHole")
-		(at 210.82 101.6 0)
+		(at 157.48 182.88 0)
 		(unit 1)
 		(exclude_from_sim yes)
@@
 		(fields_autoplaced yes)
 		(property "Reference" "H3"
-			(at 213.36 100.3299 0)
+			(at 160.02 181.6099 0)
 			(effects
 				(font
@@
 		)
 		(property "Value" "MountingHole"
-			(at 213.36 102.8699 0)
+			(at 160.02 184.1499 0)
 			(effects
 				(font
@@
 		)
 		(property "Footprint" "MountingHole:MountingHole_3.2mm_M3_DIN965_Pad"
-			(at 210.82 101.6 0)
+			(at 157.48 182.88 0)
 			(effects
 				(font
@@
 		)
 		(property "Datasheet" "~"
-			(at 210.82 101.6 0)
+			(at 157.48 182.88 0)
 			(effects
 				(font
@@
 		)
 		(property "Description" "Mounting Hole without connection"
-			(at 210.82 101.6 0)
+			(at 157.48 182.88 0)
 			(effects
 				(font
@@
 	(symbol
 		(lib_id "Mechanical:MountingHole")
-		(at 210.82 91.44 0)
+		(at 157.48 172.72 0)
 		(unit 1)
 		(exclude_from_sim yes)
@@
 		(fields_autoplaced yes)
 		(property "Reference" "H1"
-			(at 213.36 90.1699 0)
+			(at 160.02 171.4499 0)
 			(effects
 				(font
@@
 		)
 		(property "Value" "MountingHole"
-			(at 213.36 92.7099 0)
+			(at 160.02 173.9899 0)
 			(effects
 				(font
@@
 		)
 		(property "Footprint" "MountingHole:MountingHole_3.2mm_M3_DIN965_Pad"
-			(at 210.82 91.44 0)
+			(at 157.48 172.72 0)
 			(effects
 				(font
@@
 		)
 		(property "Datasheet" "~"
-			(at 210.82 91.44 0)
+			(at 157.48 172.72 0)
 			(effects
 				(font
@@
 		)
 		(property "Description" "Mounting Hole without connection"
-			(at 210.82 91.44 0)
+			(at 157.48 172.72 0)
 			(effects
 				(font
@@
 	(symbol
 		(lib_id "Mechanical:MountingHole")
-		(at 210.82 106.68 0)
+		(at 157.48 187.96 0)
 		(unit 1)
 		(exclude_from_sim yes)
@@
 		(fields_autoplaced yes)
 		(property "Reference" "H4"
-			(at 213.36 105.4099 0)
+			(at 160.02 186.6899 0)
 			(effects
 				(font
@@
 		)
 		(property "Value" "MountingHole"
-			(at 213.36 107.9499 0)
+			(at 160.02 189.2299 0)
 			(effects
 				(font
@@
 		)
 		(property "Footprint" "MountingHole:MountingHole_3.2mm_M3_DIN965_Pad"
-			(at 210.82 106.68 0)
+			(at 157.48 187.96 0)
 			(effects
 				(font
@@
 		)
 		(property "Datasheet" "~"
-			(at 210.82 106.68 0)
+			(at 157.48 187.96 0)
 			(effects
 				(font
@@
 		)
 		(property "Description" "Mounting Hole without connection"
-			(at 210.82 106.68 0)
+			(at 157.48 187.96 0)
 			(effects
 				(font
@@
 	(symbol
 		(lib_id "Mechanical:MountingHole")
-		(at 210.82 96.52 0)
+		(at 157.48 177.8 0)
 		(unit 1)
 		(exclude_from_sim yes)
@@
 		(fields_autoplaced yes)
 		(property "Reference" "H2"
-			(at 213.36 95.2499 0)
+			(at 160.02 176.5299 0)
 			(effects
 				(font
@@
 		)
 		(property "Value" "MountingHole"
-			(at 213.36 97.7899 0)
+			(at 160.02 179.0699 0)
 			(effects
 				(font
@@
 		)
 		(property "Footprint" "MountingHole:MountingHole_3.2mm_M3_DIN965_Pad"
-			(at 210.82 96.52 0)
+			(at 157.48 177.8 0)
 			(effects
 				(font
@@
 		)
 		(property "Datasheet" "~"
-			(at 210.82 96.52 0)
+			(at 157.48 177.8 0)
 			(effects
 				(font
@@
 		)
 		(property "Description" "Mounting Hole without connection"
-			(at 210.82 96.52 0)
+			(at 157.48 177.8 0)
 			(effects
 				(font
