File: hardware/opamp headphones amp with discrete transistors/opamp headphones amp with discrete transistors.kicad_sch (KiCad schematic)
At the start: 37 parts, among them J1 Conn_01x03_Pin, J2 Conn_01x03_Pin, J3 Conn_01x03_Pin, Q1 BD139, Q2 BD140, Q3 BD139, Q4 BD140, U1 NE5532

Commit message: Cosmetic cleanup in schematics, add schematic PDF exports
Other:
- title: (none) -> OpAmp Headphones Amplifier Board
- moved on the sheet: H1, H2, H3, H4
Changed lines of the file:
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@@
 	(generator_version "9.0")
 	(paper "A4")
+	(title_block
+		(title "OpAmp Headphones Amplifier Board")
+	)
 	(junction
 		(at 110.49 146.05)
@@
 	(symbol
 		(lib_id "Mechanical:MountingHole")
-		(at 177.8 152.4 0)
+		(at 147.32 193.04 0)
 		(unit 1)
 		(exclude_from_sim yes)
@@
 		(fields_autoplaced yes)
 		(property "Reference" "H2"
-			(at 180.34 151.1299 0)
+			(at 149.86 191.7699 0)
 			(effects
 				(font
@@
 		)
 		(property "Value" "MountingHole"
-			(at 180.34 153.6699 0)
+			(at 149.86 194.3099 0)
 			(effects
 				(font
@@
 		)
 		(property "Footprint" "MountingHole:MountingHole_3.2mm_M3_DIN965_Pad"
-			(at 177.8 152.4 0)
+			(at 147.32 193.04 0)
 			(effects
 				(font
@@
 		)
 		(property "Datasheet" "~"
-			(at 177.8 152.4 0)
+			(at 147.32 193.04 0)
 			(effects
 				(font
@@
 		)
 		(property "Description" "Mounting Hole without connection"
-			(at 177.8 152.4 0)
+			(at 147.32 193.04 0)
 			(effects
 				(font
@@
 	(symbol
 		(lib_id "Mechanical:MountingHole")
-		(at 190.5 152.4 0)
+		(at 160.02 193.04 0)
 		(unit 1)
 		(exclude_from_sim yes)
@@
 		(fields_autoplaced yes)
 		(property "Reference" "H4"
-			(at 193.04 151.1299 0)
+			(at 162.56 191.7699 0)
 			(effects
 				(font
@@
 		)
 		(property "Value" "MountingHole"
-			(at 193.04 153.6699 0)
+			(at 162.56 194.3099 0)
 			(effects
 				(font
@@
 		)
 		(property "Footprint" "MountingHole:MountingHole_3.2mm_M3_DIN965_Pad"
-			(at 190.5 152.4 0)
+			(at 160.02 193.04 0)
 			(effects
 				(font
@@
 		)
 		(property "Datasheet" "~"
-			(at 190.5 152.4 0)
+			(at 160.02 193.04 0)
 			(effects
 				(font
@@
 		)
 		(property "Description" "Mounting Hole without connection"
-			(at 190.5 152.4 0)
+			(at 160.02 193.04 0)
 			(effects
 				(font
@@
 	(symbol
 		(lib_id "Mechanical:MountingHole")
-		(at 177.8 146.05 0)
+		(at 147.32 186.69 0)
 		(unit 1)
 		(exclude_from_sim yes)
@@
 		(fields_autoplaced yes)
 		(property "Reference" "H1"
-			(at 180.34 144.7799 0)
+			(at 149.86 185.4199 0)
 			(effects
 				(font
@@
 		)
 		(property "Value" "MountingHole"
-			(at 180.34 147.3199 0)
+			(at 149.86 187.9599 0)
 			(effects
 				(font
@@
 		)
 		(property "Footprint" "MountingHole:MountingHole_3.2mm_M3_DIN965_Pad"
-			(at 177.8 146.05 0)
+			(at 147.32 186.69 0)
 			(effects
 				(font
@@
 		)
 		(property "Datasheet" "~"
-			(at 177.8 146.05 0)
+			(at 147.32 186.69 0)
 			(effects
 				(font
@@
 		)
 		(property "Description" "Mounting Hole without connection"
-			(at 177.8 146.05 0)
+			(at 147.32 186.69 0)
 			(effects
 				(font
@@
 	(symbol
 		(lib_id "Mechanical:MountingHole")
-		(at 190.5 146.05 0)
+		(at 160.02 186.69 0)
 		(unit 1)
 		(exclude_from_sim yes)
@@
 		(fields_autoplaced yes)
 		(property "Reference" "H3"
-			(at 193.04 144.7799 0)
+			(at 162.56 185.4199 0)
 			(effects
 				(font
@@
 		)
 		(property "Value" "MountingHole"
-			(at 193.04 147.3199 0)
+			(at 162.56 187.9599 0)
 			(effects
 				(font
@@
 		)
 		(property "Footprint" "MountingHole:MountingHole_3.2mm_M3_DIN965_Pad"
-			(at 190.5 146.05 0)
+			(at 160.02 186.69 0)
 			(effects
 				(font
@@
 		)
 		(property "Datasheet" "~"
-			(at 190.5 146.05 0)
+			(at 160.02 186.69 0)
 			(effects
 				(font
@@
 		)
 		(property "Description" "Mounting Hole without connection"
-			(at 190.5 146.05 0)
+			(at 160.02 186.69 0)
 			(effects
 				(font
